File: hardware/PCB/macrocoaster_v2.kicad_pcb (KiCad board)
At the start: 2 copper layers, 100 x 100 mm, 38 parts, among them SW1 Switch, SW10 Switch, SW11 Switch, SW13 RotaryEncoder_Switch, SW14 RotaryEncoder_Switch, SW2 Switch, SW3 Switch, SW4 Switch, SW5 Switch, SW6 Switch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

Commit message: updated kicad version
Other:
- board text added: "mm"
- board text removed: "locked"
